Commit message: fix utra6-1000 urdf model

File: utra_description/urdf/utra6_1000.urdf.xacro (robot description, xacro)
@@ -17,9 +17,9 @@
     <material name="Silver"> <color rgba="0.7 0.7 0.7 1.0"/> </material>
     <xacro:macro name="origin_joint1"> <origin xyz="0 0 0" rpy="0 0 0" /> </xacro:macro>
-    <xacro:macro name="origin_joint2"> <origin xyz="0 0 0.1174" rpy="0 0 0" /> </xacro:macro>
+    <xacro:macro name="origin_joint2"> <origin xyz="0 0 0.1175" rpy="0 0 0" /> </xacro:macro>
     <xacro:macro name="origin_joint3"> <origin xyz="0 0 0.463" rpy="0 0 0" /> </xacro:macro>
     <xacro:macro name="origin_joint4"> <origin xyz="0 0 0.4325" rpy="0 0 0" /> </xacro:macro>
-    <xacro:macro name="origin_joint5"> <origin xyz="0 -0.13993 0.1045" rpy="0 0 0" /> </xacro:macro>
-    <xacro:macro name="origin_joint6"> <origin xyz="0 -0.07507 0" rpy="0 0 0" /> </xacro:macro>
+    <xacro:macro name="origin_joint5"> <origin xyz="0 -0.1405 0.1045" rpy="0 0 0" /> </xacro:macro>
+    <xacro:macro name="origin_joint6"> <origin xyz="0 -0.0745 0" rpy="${0.5*pi} 0 0" /> </xacro:macro>
     <xacro:macro name="origin_visual_base">  <origin xyz="0 0 0" rpy="0 0 0" /> </xacro:macro>
     <xacro:macro name="origin_visual_link_1"> <origin xyz="0 0 0" rpy="0 0 0" /> </xacro:macro>
@@ -208,5 +208,5 @@
       <parent link="${prefix}link_5" />
       <child link="${prefix}link_6" />
-      <axis xyz="0 1 0" />
+      <axis xyz="0 0 1" />
       <limit lower="${joint6_lower_limit}" upper="${joint6_upper_limit}" effort="${effort_joint6}" velocity="3.14" />
       <dynamics damping="${damping_joint6}" friction="${friction_joint6}" />
