Commit message: fix opti6-800 urdf model

File: utra_description/urdf/opti6_800.urdf.xacro (robot description, xacro)
@@ -5,5 +5,5 @@
     Contributers:
   -->
-  <xacro:macro name="opti6_urdf" params="prefix
+  <xacro:macro name="opti6_800_urdf" params="prefix
     joint1_lower_limit:=${-2.0*pi} joint1_upper_limit:=${2.0*pi}
     joint2_lower_limit:=${-2.0*pi} joint2_upper_limit:=${2.0*pi}
@@ -18,6 +18,5 @@
     <xacro:macro name="origin_joint1"> <origin xyz="0 0 0" rpy="0 0 0" /> </xacro:macro>
     <xacro:macro name="origin_joint2"> <origin xyz="0 0 0.278" rpy="0 0 0" /> </xacro:macro>
-    <xacro:macro name="_origin_joint3"> <origin xyz="0 0 0.1993" rpy="0 0 0" /> </xacro:macro>
-    <xacro:macro name="origin_joint3"> <origin xyz="0 0 0.1507" rpy="0 0 0" /> </xacro:macro>
+    <xacro:macro name="origin_joint3"> <origin xyz="0 0 0.35" rpy="0 0 0" /> </xacro:macro>
     <xacro:macro name="origin_joint4"> <origin xyz="0 0 0.1677" rpy="0 0 0" /> </xacro:macro>
     <xacro:macro name="origin_joint5"> <origin xyz="0 0 0.1393" rpy="0 0 0" /> </xacro:macro>
@@ -133,28 +132,7 @@
       </collision>
     </link>
-    <joint name="${prefix}joint3_" type="fixed">
-      <xacro:_origin_joint3/>
-      <parent link="${prefix}link_2" />
-      <child link="${prefix}link_3_" />
-    </joint>
-    <link name="${prefix}link_3_">
-      <inertial>
-        <xacro:origin_inertial_link_3/>
-        <mass value="${mass_link_3}" />
-        <xacro:inertia_link_3/>
-      </inertial>
-      <visual>
-        <xacro:origin_visual_link_3/>
-        <geometry> <mesh filename="package://utra_description/meshes/opti6_800/visual/link3.STL" /> </geometry>
-        <material name="Silver" />
-      </visual>
-      <collision>
-        <xacro:origin_visual_link_3/>
-        <geometry> <mesh filename="package://utra_description/meshes/opti6_800/visual/link3.STL" /> </geometry>
-      </collision>
-    </link>
     <joint name="${prefix}joint3" type="revolute">
       <xacro:origin_joint3/>
-      <parent link="${prefix}link_3_" />
+      <parent link="${prefix}link_2" />
       <child link="${prefix}link_3" />
       <axis xyz="0 -1 0" />
@@ -170,10 +148,10 @@
       <visual>
         <xacro:origin_visual_link_3/>
-        <geometry> <mesh filename="package://utra_description/meshes/opti6_800/visual/link4.STL" /> </geometry>
+        <geometry> <mesh filename="package://utra_description/meshes/opti6_800/visual/link3.STL" /> </geometry>
         <material name="Silver" />
       </visual>
       <collision>
         <xacro:origin_visual_link_3/>
-        <geometry> <mesh filename="package://utra_description/meshes/opti6_800/visual/link4.STL" /> </geometry>
+        <geometry> <mesh filename="package://utra_description/meshes/opti6_800/visual/link3.STL" /> </geometry>
       </collision>
     </link>
@@ -194,10 +172,10 @@
       <visual>
         <xacro:origin_visual_link_4/>
-        <geometry> <mesh filename="package://utra_description/meshes/opti6_800/visual/link5.STL" /> </geometry>
+        <geometry> <mesh filename="package://utra_description/meshes/opti6_800/visual/link4.STL" /> </geometry>
         <material name="Silver" />
       </visual>
       <collision>
         <xacro:origin_visual_link_4/>
-        <geometry> <mesh filename="package://utra_description/meshes/opti6_800/visual/link5.STL" /> </geometry>
+        <geometry> <mesh filename="package://utra_description/meshes/opti6_800/visual/link4.STL" /> </geometry>
       </collision>
     </link>
@@ -218,10 +196,10 @@
       <visual>
         <xacro:origin_visual_link_5/>
-        <geometry> <mesh filename="package://utra_description/meshes/opti6_800/visual/link6.STL" /> </geometry>
+        <geometry> <mesh filename="package://utra_description/meshes/opti6_800/visual/link5.STL" /> </geometry>
         <material name="Silver" />
       </visual>
       <collision>
         <xacro:origin_visual_link_5/>
-        <geometry> <mesh filename="package://utra_description/meshes/opti6_800/visual/link6.STL" /> </geometry>
+        <geometry> <mesh filename="package://utra_description/meshes/opti6_800/visual/link5.STL" /> </geometry>
       </collision>
     </link>
@@ -242,10 +220,10 @@
       <visual>
         <xacro:origin_visual_link_6/>
-        <geometry> <mesh filename="package://utra_description/meshes/opti6_800/visual/link7.STL" /> </geometry>
+        <geometry> <mesh filename="package://utra_description/meshes/opti6_800/visual/link6.STL" /> </geometry>
         <material name="Silver" />
       </visual>
       <collision>
         <xacro:origin_visual_link_6/>
-        <geometry> <mesh filename="package://utra_description/meshes/opti6_800/visual/link7.STL" /> </geometry>
+        <geometry> <mesh filename="package://utra_description/meshes/opti6_800/visual/link6.STL" /> </geometry>
       </collision>
     </link>

File: utra_description/urdf/opti6_800_common.gazebo.xacro (robot description, xacro)
@@ -3,5 +3,5 @@
   <gazebo>
     <plugin name="gazebo_ros_control" filename="libgazebo_ros_control.so">
-      <robotNamespace>/opti6</robotNamespace>
+      <robotNamespace>/opti6_800</robotNamespace>
       <robotSimType>gazebo_ros_control/DefaultRobotHWSim</robotSimType>
       <legacyModeNS>true</legacyModeNS>

File: utra_description/urdf/opti6_800_robot.urdf.xacro (robot description, xacro)
@@ -1,4 +1,4 @@
 <?xml version='1.0' encoding='utf-8'?>
-<robot xmlns:xacro="http://ros.org/wiki/xacro" name="opti6">
+<robot xmlns:xacro="http://ros.org/wiki/xacro" name="opti6_800">
   <xacro:arg name="prefix" default=""/>
   <xacro:arg name="ros_namespace" default="utra"/>
@@ -17,5 +17,5 @@
     </joint>
     <xacro:if value="$(arg limited)">
-      <xacro:opti6_urdf prefix="$(arg prefix)"
+      <xacro:opti6_800_urdf prefix="$(arg prefix)"
         joint1_lower_limit="${-2.0*pi}" joint1_upper_limit="${2.0*pi}"
         joint2_lower_limit="${-2.0*pi}" joint2_upper_limit="${2.0*pi}"
@@ -26,5 +26,5 @@
     </xacro:if>
     <xacro:unless value="$(arg limited)">
-      <xacro:opti6_urdf prefix="$(arg prefix)"/>
+      <xacro:opti6_800_urdf prefix="$(arg prefix)"/>
     </xacro:unless>
   <xacro:include filename="$(find utra_description)/urdf/transmission.xacro" />

File: utra_description/urdf/opti6_800_robot_gripper.urdf.xacro (robot description, xacro)
@@ -1,4 +1,4 @@
 <?xml version='1.0' encoding='utf-8'?>
-<robot xmlns:xacro="http://ros.org/wiki/xacro" name="opti6">
+<robot xmlns:xacro="http://ros.org/wiki/xacro" name="opti6_800">
   <xacro:arg name="prefix" default=""/>
   <xacro:arg name="ros_namespace" default="utra"/>
@@ -30,5 +30,5 @@
     </joint>
     <xacro:if value="$(arg limited)">
-      <xacro:opti6_urdf prefix="$(arg prefix)"
+      <xacro:opti6_800_urdf prefix="$(arg prefix)"
         joint1_lower_limit="${-2.0*pi}" joint1_upper_limit="${2.0*pi}"
         joint2_lower_limit="${-2.0*pi}" joint2_upper_limit="${2.0*pi}"
@@ -39,5 +39,5 @@
     </xacro:if>
     <xacro:unless value="$(arg limited)">
-      <xacro:opti6_urdf prefix="$(arg prefix)"/>
+      <xacro:opti6_800_urdf prefix="$(arg prefix)"/>
     </xacro:unless>
   <xacro:include filename="$(find utra_description)/urdf/transmission.xacro" />

File: utra_description/urdf/opti6_800_robot_vacuum_gripper.urdf.xacro (robot description, xacro)
@@ -1,4 +1,4 @@
 <?xml version='1.0' encoding='utf-8'?>
-<robot xmlns:xacro="http://ros.org/wiki/xacro" name="opti6">
+<robot xmlns:xacro="http://ros.org/wiki/xacro" name="opti6_800">
   <xacro:arg name="prefix" default=""/>
   <xacro:arg name="ros_namespace" default="utra"/>
@@ -17,5 +17,5 @@
     </joint>
     <xacro:if value="$(arg limited)">
-      <xacro:opti6_urdf prefix="$(arg prefix)"
+      <xacro:opti6_800_urdf prefix="$(arg prefix)"
         joint1_lower_limit="${-2.0*pi}" joint1_upper_limit="${2.0*pi}"
         joint2_lower_limit="${-2.0*pi}" joint2_upper_limit="${2.0*pi}"
@@ -26,5 +26,5 @@
     </xacro:if>
     <xacro:unless value="$(arg limited)">
-      <xacro:opti6_urdf prefix="$(arg prefix)"/>
+      <xacro:opti6_800_urdf prefix="$(arg prefix)"/>
     </xacro:unless>
   <xacro:include filename="$(find utra_description)/urdf/transmission.xacro" />

File: utra_description/urdf/opti7_800.urdf.xacro (robot description, xacro)
@@ -5,5 +5,5 @@
     Contributers:
   -->
-  <xacro:macro name="opti7_urdf" params="prefix
+  <xacro:macro name="opti7_800_urdf" params="prefix
     joint1_lower_limit:=${-2.0*pi} joint1_upper_limit:=${2.0*pi}
     joint2_lower_limit:=${-2.0*pi} joint2_upper_limit:=${2.0*pi}
