Commit message: fix opti7-800 urdf model

File: utra_description/urdf/opti7_800.urdf.xacro (robot description, xacro)
@@ -85,10 +85,10 @@
       <visual>
         <xacro:origin_visual_base/>
-        <geometry> <mesh filename="package://utra_description/meshes/opti6_800/visual/base.STL" /> </geometry>
+        <geometry> <mesh filename="package://utra_description/meshes/opti7_800/visual/base.STL" /> </geometry>
         <material name="Silver" />
       </visual>
       <collision>
         <xacro:origin_visual_base/>
-        <geometry> <mesh filename="package://utra_description/meshes/opti6_800/visual/base.STL" /> </geometry>
+        <geometry> <mesh filename="package://utra_description/meshes/opti7_800/visual/base.STL" /> </geometry>
       </collision>
     </link>
@@ -109,10 +109,10 @@
       <visual>
         <xacro:origin_visual_link_1/>
-        <geometry> <mesh filename="package://utra_description/meshes/opti6_800/visual/link1.STL" /> </geometry>
+        <geometry> <mesh filename="package://utra_description/meshes/opti7_800/visual/link1.STL" /> </geometry>
         <material name="Silver" />
       </visual>
       <collision>
         <xacro:origin_visual_link_1/>
-        <geometry> <mesh filename="package://utra_description/meshes/opti6_800/visual/link1.STL" /> </geometry>
+        <geometry> <mesh filename="package://utra_description/meshes/opti7_800/visual/link1.STL" /> </geometry>
       </collision>
     </link>
@@ -133,10 +133,10 @@
       <visual>
         <xacro:origin_visual_link_2/>
-        <geometry> <mesh filename="package://utra_description/meshes/opti6_800/visual/link2.STL" /> </geometry>
+        <geometry> <mesh filename="package://utra_description/meshes/opti7_800/visual/link2.STL" /> </geometry>
         <material name="Silver" />
       </visual>
       <collision>
         <xacro:origin_visual_link_2/>
-        <geometry> <mesh filename="package://utra_description/meshes/opti6_800/visual/link2.STL" /> </geometry>
+        <geometry> <mesh filename="package://utra_description/meshes/opti7_800/visual/link2.STL" /> </geometry>
       </collision>
     </link>
@@ -157,10 +157,10 @@
       <visual>
         <xacro:origin_visual_link_3/>
-        <geometry> <mesh filename="package://utra_description/meshes/opti6_800/visual/link3.STL" /> </geometry>
+        <geometry> <mesh filename="package://utra_description/meshes/opti7_800/visual/link3.STL" /> </geometry>
         <material name="Silver" />
       </visual>
       <collision>
         <xacro:origin_visual_link_3/>
-        <geometry> <mesh filename="package://utra_description/meshes/opti6_800/visual/link3.STL" /> </geometry>
+        <geometry> <mesh filename="package://utra_description/meshes/opti7_800/visual/link3.STL" /> </geometry>
       </collision>
     </link>
@@ -181,14 +181,14 @@
       <visual>
         <xacro:origin_visual_link_4/>
-        <geometry> <mesh filename="package://utra_description/meshes/opti6_800/visual/link4.STL" /> </geometry>
+        <geometry> <mesh filename="package://utra_description/meshes/opti7_800/visual/link4.STL" /> </geometry>
         <material name="Silver" />
       </visual>
       <collision>
         <xacro:origin_visual_link_4/>
-        <geometry> <mesh filename="package://utra_description/meshes/opti6_800/visual/link4.STL" /> </geometry>
+        <geometry> <mesh filename="package://utra_description/meshes/opti7_800/visual/link4.STL" /> </geometry>
       </collision>
     </link>
     <joint name="${prefix}joint5" type="revolute">
-      <xacro:origin_joint4/>
+      <xacro:origin_joint5/>
       <parent link="${prefix}link_4" />
       <child link="${prefix}link_5" />
@@ -205,10 +205,10 @@
       <visual>
         <xacro:origin_visual_link_5/>
-        <geometry> <mesh filename="package://utra_description/meshes/opti6_800/visual/link5.STL" /> </geometry>
+        <geometry> <mesh filename="package://utra_description/meshes/opti7_800/visual/link5.STL" /> </geometry>
         <material name="Silver" />
       </visual>
       <collision>
         <xacro:origin_visual_link_5/>
-        <geometry> <mesh filename="package://utra_description/meshes/opti6_800/visual/link5.STL" /> </geometry>
+        <geometry> <mesh filename="package://utra_description/meshes/opti7_800/visual/link5.STL" /> </geometry>
       </collision>
     </link>
@@ -229,10 +229,10 @@
       <visual>
         <xacro:origin_visual_link_6/>
-        <geometry> <mesh filename="package://utra_description/meshes/opti6_800/visual/link6.STL" /> </geometry>
+        <geometry> <mesh filename="package://utra_description/meshes/opti7_800/visual/link6.STL" /> </geometry>
         <material name="Silver" />
       </visual>
       <collision>
         <xacro:origin_visual_link_6/>
-        <geometry> <mesh filename="package://utra_description/meshes/opti6_800/visual/link6.STL" /> </geometry>
+        <geometry> <mesh filename="package://utra_description/meshes/opti7_800/visual/link6.STL" /> </geometry>
       </collision>
     </link>
@@ -253,10 +253,10 @@
       <visual>
         <xacro:origin_visual_link_7/>
-        <geometry> <mesh filename="package://utra_description/meshes/opti6_800/visual/link7.STL" /> </geometry>
+        <geometry> <mesh filename="package://utra_description/meshes/opti7_800/visual/link7.STL" /> </geometry>
         <material name="Silver" />
       </visual>
       <collision>
         <xacro:origin_visual_link_7/>
-        <geometry> <mesh filename="package://utra_description/meshes/opti6_800/visual/link7.STL" /> </geometry>
+        <geometry> <mesh filename="package://utra_description/meshes/opti7_800/visual/link7.STL" /> </geometry>
       </collision>
     </link>

File: utra_description/urdf/opti7_800_common.gazebo.xacro (robot description, xacro)
@@ -3,5 +3,5 @@
   <gazebo>
     <plugin name="gazebo_ros_control" filename="libgazebo_ros_control.so">
-      <robotNamespace>/opti7</robotNamespace>
+      <robotNamespace>/opti7_800</robotNamespace>
       <robotSimType>gazebo_ros_control/DefaultRobotHWSim</robotSimType>
       <legacyModeNS>true</legacyModeNS>

File: utra_description/urdf/opti7_800_robot.urdf.xacro (robot description, xacro)
@@ -1,4 +1,4 @@
 <?xml version='1.0' encoding='utf-8'?>
-<robot xmlns:xacro="http://ros.org/wiki/xacro" name="opti7">
+<robot xmlns:xacro="http://ros.org/wiki/xacro" name="opti7_800">
   <xacro:arg name="prefix" default=""/>
   <xacro:arg name="ros_namespace" default="utra"/>
@@ -17,5 +17,5 @@
     </joint>
     <xacro:if value="$(arg limited)">
-      <xacro:opti7_urdf prefix="$(arg prefix)"
+      <xacro:opti7_800_urdf prefix="$(arg prefix)"
         joint1_lower_limit="${-2.0*pi}" joint1_upper_limit="${2.0*pi}"
         joint2_lower_limit="${-2.0*pi}" joint2_upper_limit="${2.0*pi}"
@@ -27,5 +27,5 @@
     </xacro:if>
     <xacro:unless value="$(arg limited)">
-      <xacro:opti7_urdf prefix="$(arg prefix)"/>
+      <xacro:opti7_800_urdf prefix="$(arg prefix)"/>
     </xacro:unless>
   <xacro:include filename="$(find utra_description)/urdf/transmission.xacro" />

File: utra_description/urdf/opti7_800_robot_gripper.urdf.xacro (robot description, xacro)
@@ -1,4 +1,4 @@
 <?xml version='1.0' encoding='utf-8'?>
-<robot xmlns:xacro="http://ros.org/wiki/xacro" name="opti7">
+<robot xmlns:xacro="http://ros.org/wiki/xacro" name="opti7_800">
   <xacro:arg name="prefix" default=""/>
   <xacro:arg name="ros_namespace" default="utra"/>
@@ -30,5 +30,5 @@
     </joint>
     <xacro:if value="$(arg limited)">
-      <xacro:opti7_urdf prefix="$(arg prefix)"
+      <xacro:opti7_800_urdf prefix="$(arg prefix)"
         joint1_lower_limit="${-2.0*pi}" joint1_upper_limit="${2.0*pi}"
         joint2_lower_limit="${-2.0*pi}" joint2_upper_limit="${2.0*pi}"
@@ -40,5 +40,5 @@
     </xacro:if>
     <xacro:unless value="$(arg limited)">
-      <xacro:opti7_urdf prefix="$(arg prefix)"/>
+      <xacro:opti7_800_urdf prefix="$(arg prefix)"/>
     </xacro:unless>
   <xacro:include filename="$(find utra_description)/urdf/transmission.xacro" />

File: utra_description/urdf/opti7_800_robot_vacuum_gripper.urdf.xacro (robot description, xacro)
@@ -1,4 +1,4 @@
 <?xml version='1.0' encoding='utf-8'?>
-<robot xmlns:xacro="http://ros.org/wiki/xacro" name="opti7">
+<robot xmlns:xacro="http://ros.org/wiki/xacro" name="opti7_800">
   <xacro:arg name="prefix" default=""/>
   <xacro:arg name="ros_namespace" default="utra"/>
@@ -17,5 +17,5 @@
     </joint>
     <xacro:if value="$(arg limited)">
-      <xacro:opti7_urdf prefix="$(arg prefix)"
+      <xacro:opti7_800_urdf prefix="$(arg prefix)"
         joint1_lower_limit="${-2.0*pi}" joint1_upper_limit="${2.0*pi}"
         joint2_lower_limit="${-2.0*pi}" joint2_upper_limit="${2.0*pi}"
@@ -27,5 +27,5 @@
     </xacro:if>
     <xacro:unless value="$(arg limited)">
-      <xacro:opti7_urdf prefix="$(arg prefix)"/>
+      <xacro:opti7_800_urdf prefix="$(arg prefix)"/>
     </xacro:unless>
   <xacro:include filename="$(find utra_description)/urdf/transmission.xacro" />
