Commit message: add link_tcp on gripper model

File: utra_description/urdf/utra6_1000_robot_gripper.urdf.xacro (robot description, xacro)
@@ -16,4 +16,16 @@
       <child link = "$(arg prefix)base_link" />
       <origin xyz="0 0 0" rpy="0 0 0" />
+    </joint>
+    <link name="$(arg prefix)link_tcp" />
+    <joint
+      name="$(arg prefix)joint_tcp"
+      type="fixed">
+      <origin
+        xyz="0 -0.18 0"
+        rpy="0 0 0" />
+      <parent
+        link="$(arg prefix)link_6" />
+      <child
+        link="$(arg prefix)link_tcp" />
     </joint>
     <xacro:if value="$(arg limited)">

File: utra_description/urdf/utra6_550_robot_gripper.urdf.xacro (robot description, xacro)
@@ -16,4 +16,16 @@
       <child link = "$(arg prefix)base_link" />
       <origin xyz="0 0 0" rpy="0 0 0" />
+    </joint>
+    <link name="$(arg prefix)link_tcp" />
+    <joint
+      name="$(arg prefix)joint_tcp"
+      type="fixed">
+      <origin
+        xyz="0 -0.18 0"
+        rpy="0 0 0" />
+      <parent
+        link="$(arg prefix)link_6" />
+      <child
+        link="$(arg prefix)link_tcp" />
     </joint>
     <xacro:if value="$(arg limited)">

File: utra_description/urdf/utra6_850_robot_gripper.urdf.xacro (robot description, xacro)
@@ -16,4 +16,16 @@
       <child link = "$(arg prefix)base_link" />
       <origin xyz="0 0 0" rpy="0 0 0" />
+    </joint>
+    <link name="$(arg prefix)link_tcp" />
+    <joint
+      name="$(arg prefix)joint_tcp"
+      type="fixed">
+      <origin
+        xyz="0 0 0.18"
+        rpy="0 0 0" />
+      <parent
+        link="$(arg prefix)link_6" />
+      <child
+        link="$(arg prefix)link_tcp" />
     </joint>
     <xacro:if value="$(arg limited)">

Commit message: update moveit

File: utra_description/urdf/utra6_1000_robot_gripper.urdf.xacro (robot description, xacro)
@@ -23,5 +23,5 @@
       type="fixed">
       <origin
-        xyz="0 -0.18 0"
+        xyz="0 0 0.18"
         rpy="0 0 0" />
       <parent
@@ -70,5 +70,5 @@
         <parent link="$(arg prefix)link_6"/>
         <child link="$(arg prefix)d435i"/>
-        <origin xyz="0 0 0" rpy="0 -${pi/2} ${pi/2}"/>
+        <origin xyz="0 0 0" rpy="0 0 ${pi/2}"/>
     </joint>
     <xacro:if value="$(arg add_gripper)" >
@@ -83,5 +83,5 @@
           <xacro:include filename="$(find utra_gripper)/urdf/gripper.urdf.xacro" />
           <xacro:gripper prefix="$(arg prefix)" parent="$(arg prefix)link_6" >
-            <origin xyz="0 0 0" rpy="1.571 1.571 0"/>
+            <origin xyz="0 0 0" rpy="0 0 ${pi/2}"/>
           </xacro:gripper>
       </xacro:if>

File: utra_description/urdf/utra6_1000_robot_vacuum_gripper.urdf.xacro (robot description, xacro)
@@ -39,5 +39,5 @@
   <xacro:include filename="$(find utra_vacuum_gripper)/urdf/vacuum_gripper.urdf.xacro" />
   <xacro:vacuum_gripper prefix="$(arg prefix)" parent="$(arg prefix)link_6" >
-        <origin xyz="0 0.008 0" rpy="1.57 0 0"/>
+      <origin xyz="0 0 -0.008" rpy="0 0 0"/>
   </xacro:vacuum_gripper>
 </robot>

File: utra_description/urdf/utra6_550_robot_gripper.urdf.xacro (robot description, xacro)
@@ -23,5 +23,5 @@
       type="fixed">
       <origin
-        xyz="0 -0.18 0"
+        xyz="0 0 0.18"
         rpy="0 0 0" />
       <parent
@@ -70,5 +70,5 @@
         <parent link="$(arg prefix)link_6"/>
         <child link="$(arg prefix)d435i"/>
-        <origin xyz="0 0 0" rpy="0 -${pi/2} ${pi/2}"/>
+        <origin xyz="0 0 0" rpy="0 0 ${pi/2}"/>
     </joint>
     <xacro:if value="$(arg add_gripper)" >
@@ -83,5 +83,5 @@
           <xacro:include filename="$(find utra_gripper)/urdf/gripper.urdf.xacro" />
           <xacro:gripper prefix="$(arg prefix)" parent="$(arg prefix)link_6" >
-            <origin xyz="0 0 0" rpy="1.571 1.571 0"/>
+            <origin xyz="0 0 0" rpy="0 0 ${pi/2}"/>
           </xacro:gripper>
       </xacro:if>

File: utra_description/urdf/utra6_550_robot_vacuum_gripper.urdf.xacro (robot description, xacro)
@@ -38,5 +38,5 @@
   <xacro:include filename="$(find utra_vacuum_gripper)/urdf/vacuum_gripper.urdf.xacro" />
   <xacro:vacuum_gripper prefix="$(arg prefix)" parent="$(arg prefix)link_6" >
-        <origin xyz="0 0.008 0" rpy="1.57 0 0"/>
+        <origin xyz="0 0 -0.008" rpy="0 0 0"/>
     </xacro:vacuum_gripper>
 </robot>

File: utra_description/urdf/utra6_850_robot_gripper.urdf.xacro (robot description, xacro)
@@ -83,5 +83,5 @@
           <xacro:include filename="$(find utra_gripper)/urdf/gripper.urdf.xacro" />
           <xacro:gripper prefix="$(arg prefix)" parent="$(arg prefix)link_6" >
-            <origin xyz="0 0 0" rpy="0 0 1.571"/>
+            <origin xyz="0 0 0" rpy="0 0 ${pi/2}"/>
           </xacro:gripper>
       </xacro:if>

File: utra_description/urdf/utra6_850_robot_vacuum_gripper.urdf.xacro (robot description, xacro)
@@ -39,5 +39,5 @@
   <xacro:include filename="$(find utra_vacuum_gripper)/urdf/vacuum_gripper.urdf.xacro" />
   <xacro:vacuum_gripper prefix="$(arg prefix)" parent="$(arg prefix)link_6" >
-        <origin xyz="0 0 -0.008" rpy="0 0 0"/>
-    </xacro:vacuum_gripper>
+      <origin xyz="0 0 -0.008" rpy="0 0 0"/>
+  </xacro:vacuum_gripper>
 </robot>
